File: circuits/nodemcu_based/nodemcu_based.kicad_pcb (KiCad board)
At the start: 2 copper layers, 77.8 x 71.2 mm, 25 parts, among them J2 Temp/Hum, J3 Lux, J4 CO2, SW1 SW_Push_DPDT, U1 ESP32_NODEMCU, U2 INMP441

Commit message: Tinggal Latex/PDF nya
Parts:
- removed J3: Lux, Connector_PinSocket_2.54mm:PinSocket_1x04_P2.54mm_Vertical
- added J1: Lux, Connector_PinSocket_2.54mm:PinSocket_1x05_P2.54mm_Vertical, F.Cu at (131.1, 124.6)
Routing:
- net GND: track 144.2 -> 100.3 mm, vias 7 -> 5
- net VDD: track 192.4 -> 181.5 mm, vias 6 -> 7
- net I2C_SCL: track 59.3 -> 50.0 mm
- net I2C_SDA: track 46.8 -> 46.6 mm, vias 3 -> 1

Commit message: Nyicil Dokumen
Parts:
- R10, R6, R7, R8, R9: value 220 -> 560
Routing:
- net +BATT: track 70.7 -> 69.5 mm
