File: circuits/nodemcu_based/nodemcu_based.kicad_sch (KiCad schematic)
At the start: 26 parts, among them J1 UART, J2 Temp/Hum, J3 Lux, J4 CO2, SW1 SW_Push_DPDT, U1 ESP32_NODEMCU, U2 INMP441

Commit message: NOdeMCU Smarthome
Parts:
- removed J1: UART, symbol Connector:Conn_01x04_Pin
- BT1, BT2: footprint (none) -> Battery:BatteryHolder_MPD_BH-18650-PC2
- D1: footprint (none) -> Diode_THT:D_DO-201_P15.24mm_Horizontal
- D2, D3, D4, D5, D6: footprint (none) -> LED_SMD:LED_0805_2012Metric_Pad1.15x1.40mm_HandSolder
- J2, J3: footprint (none) -> Connector_PinSocket_2.54mm:PinSocket_1x04_P2.54mm_Vertical
- J4: footprint (none) -> Connector_PinHeader_2.54mm:PinHeader_1x03_P2.54mm_Vertical
- R1, R10, R11, R2, R3, R4, R5, R6, R7, R8, R9: footprint (none) -> Resistor_SMD:R_0805_2012Metric_Pad1.20x1.40mm_HandSolder
- SW1: footprint (none) -> Button_Switch_THT:SW_Push_2P2T_Toggle_CK_PVA2OAH5xxxxxxV2
- U1: footprint MODULE_ESP32_NODEMCU -> ESP32_NODEMCU:MODULE_ESP32_NODEMCU
- U2: footprint (none) -> INMP441:INMP441
Connections:
- net GND: now also J2.2 (Pin_2), J3.2 (Pin_2); no longer J2.3 (Pin_3), J3.3 (Pin_3)
- net I2C_SCL: now also J2.4 (Pin_4), J3.4 (Pin_4); no longer J2.1 (Pin_1), J3.1 (Pin_1)
- net I2C_SDA: now also J2.3 (Pin_3), J3.3 (Pin_3); no longer J2.2 (Pin_2), J3.2 (Pin_2)
- net VCC: now also D1.1 (K), R2.1
- net VDD: now also J2.1 (Pin_1), J3.1 (Pin_1); no longer D1.1 (K), J2.4 (Pin_4), J3.4 (Pin_4), R2.1
- net RXD: no longer names the net of U1.J4_5 (RXD)
- net TXD: no longer names the net of U1.J4_4 (TXD)
- no-connect marks 18 -> 22
Other:
- moved on the sheet: BT1, BT2, D1, J2, J3, J4, R1, R11, R2, SW1, U2

Commit message: Tinggal Latex/PDF nya
Parts:
- removed J3: Lux, Connector_PinSocket_2.54mm:PinSocket_1x04_P2.54mm_Vertical, symbol Connector:Conn_01x04_Socket
- added J1: Lux, Connector_PinSocket_2.54mm:PinSocket_1x05_P2.54mm_Vertical, symbol Connector:Conn_01x05_Socket
Connections:
- net GND: now also J1.2 (Pin_2)
- net I2C_SCL: now also J1.4 (Pin_4)
- net I2C_SDA: now also J1.3 (Pin_3)
- net VDD: now also J1.1 (Pin_1)
- no-connect marks 22 -> 23
Changed lines of the file:
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@@
   (no_connect (at 96.52 82.55))
   (no_connect (at 96.52 105.41))
+  (no_connect (at 186.69 91.44))
   (no_connect (at 137.16 82.55))
   (no_connect (at 96.52 118.11))
@@
         (path "/64165e7f-57e2-481c-9304-1c163cb4991b"
           (reference "D2") (unit 1)
+        )
+      )
+    )
+  )
+  (symbol (lib_id "Connector:Conn_01x05_Socket") (at 191.77 86.36 270) (mirror x) (unit 1)
+    (in_bom yes) (on_board yes) (dnp no)
+    (property "Reference" "J1" (at 191.77 82.55 90)
+      (effects (font (size 1.27 1.27)))
+    )
+    (property "Value" "Lux" (at 191.77 85.09 90)
+      (effects (font (size 1.27 1.27)))
+    )
+    (property "Footprint" "Connector_PinSocket_2.54mm:PinSocket_1x05_P2.54mm_Vertical" (at 191.77 86.36 0)
+      (effects (font (size 1.27 1.27)) hide)
+    )
+    (property "Datasheet" "~" (at 191.77 86.36 0)
+      (effects (font (size 1.27 1.27)) hide)
+    )
+    (pin "1")
+    (pin "2")
+    (pin "3")
+    (pin "4")
+    (pin "5")
+    (instances
+      (project "nodemcu_based"
+        (path "/64165e7f-57e2-481c-9304-1c163cb4991b"
+          (reference "J1") (unit 1)
         )
       )
@@
         )
       )
-    )
-  )
-  (symbol (lib_id "Connector:Conn_01x04_Socket") (at 194.31 86.36 270) (mirror x) (unit 1)
-    (in_bom yes) (on_board yes) (dnp no)
-    (property "Reference" "J3" (at 193.04 82.55 90)
-      (effects (font (size 1.27 1.27)))
-    )
-    (property "Value" "Lux" (at 193.04 85.09 90)
-      (effects (font (size 1.27 1.27)))
-    )
-    (property "Footprint" "Connector_PinSocket_2.54mm:PinSocket_1x04_P2.54mm_Vertical" (at 194.31 86.36 0)
-      (effects (font (size 1.27 1.27)) hide)
-    )
-    (property "Datasheet" "~" (at 194.31 86.36 0)
-      (effects (font (size 1.27 1.27)) hide)
-    )
-    (pin "1")
-    (pin "2")
-    (pin "3")
-    (pin "4")
-    (instances
-      (project "nodemcu_based"
-        (path "/64165e7f-57e2-481c-9304-1c163cb4991b"
-          (reference "J3") (unit 1)
-        )
-      )

Commit message: Nyicil Dokumen
Parts:
- R10, R6, R7, R8, R9: value 220 -> 560
Changed lines of the file:
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@@
       (effects (font (size 1.27 1.27)) (justify left))
     )
-    (property "Value" "220" (at 185.42 57.15 90)
+    (property "Value" "560" (at 185.42 57.15 90)
       (effects (font (size 1.27 1.27)) (justify left))
     )
@@
       (effects (font (size 1.27 1.27)) (justify left))
     )
-    (property "Value" "220" (at 200.66 57.15 90)
+    (property "Value" "560" (at 200.66 57.15 90)
       (effects (font (size 1.27 1.27)) (justify left))
     )
@@
       (effects (font (size 1.27 1.27)) (justify left))
     )
-    (property "Value" "220" (at 208.28 57.15 90)
+    (property "Value" "560" (at 208.28 57.15 90)
       (effects (font (size 1.27 1.27)) (justify left))
     )
@@
       (effects (font (size 1.27 1.27)) (justify left))
     )
-    (property "Value" "220" (at 179.07 57.15 90)
+    (property "Value" "560" (at 179.07 57.15 90)
       (effects (font (size 1.27 1.27)) (justify left))
     )
@@
       (effects (font (size 1.27 1.27)) (justify left))
     )
-    (property "Value" "220" (at 193.04 57.15 90)
-      (effects (font (size 1.27 1.27)) (justify left))
-    )
+    (property "Value" "560" (at 193.04 57.15 90)
+      (effects (font (size 1.27 1.27)) (justify left))
+    )
